File: pcb/SUAD.kicad_pcb (KiCad board)
At the start: 2 copper layers, 100 x 102.5 mm, 89 parts, among them Q1 AO3401A, Q2 AO3401A, Q3 AO3401A, SW1 SW_MEC_5E, SW10 SW_MEC_5E, SW11 SW_MEC_5E, SW12 SW_MEC_5E, SW13 SW_DIP_x06, SW2 SW_MEC_5E, SW3 SW_MEC_5E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

Commit message: workflow trigger
Parts:
- moved C2 2.00 mm to (185.5, 155.0)
- moved C3 2.00 mm to (179.5, 155.0)
- moved C4 2.00 mm to (173.5, 155.0)
- moved C5 2.00 mm to (167.5, 155.0)
- moved C6 2.00 mm to (161.0, 155.0)
- moved D26 2.00 mm to (160.5, 150.0)
- moved D27 2.00 mm to (167.0, 150.0)
- moved D28 2.00 mm to (173.0, 150.0)
- moved D29 2.00 mm to (179.0, 150.0)
- moved D30 2.00 mm to (185.0, 150.0)
- moved D31 2.00 mm to (160.5, 144.0)
- moved D32 2.00 mm to (167.0, 144.0)
- moved D33 2.00 mm to (173.0, 144.0)
- moved D34 2.00 mm to (179.0, 144.0)
- moved D35 2.00 mm to (185.0, 144.0)
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Other:
- board size 100 x 102.5 mm -> 100 x 100.5 mm

Commit message: workflow trigger
Other:
- board size 100 x 100.5 mm -> 100 x 100 mm
Changed lines of the file:
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@@
   (gr_line (start 110.75 122) (end 209.25 122) (layer "F.SilkS") (width 0.15))
   (gr_line (start 146 94) (end 146 122) (layer "F.SilkS") (width 0.15))
-  (gr_line (start 156 122) (end 156 159) (layer "F.SilkS") (width 0.15))
+  (gr_line (start 156 122) (end 156 156.5) (layer "F.SilkS") (width 0.15))
   (gr_line (start 175 94) (end 175 122) (layer "F.SilkS") (width 0.15))
-  (gr_arc (start 115 158) (mid 111.464466 156.535534) (end 110 153) (layer "Edge.Cuts") (width 0.1))
-  (gr_line (start 205 158) (end 115 158) (layer "Edge.Cuts") (width 0.1))
-  (gr_line (start 210 153) (end 210 117.5) (layer "Edge.Cuts") (width 0.1))
+  (gr_arc (start 115 157.5) (mid 111.464466 156.035534) (end 110 152.5) (layer "Edge.Cuts") (width 0.1))
+  (gr_line (start 205 157.5) (end 115 157.5) (layer "Edge.Cuts") (width 0.1))
+  (gr_line (start 210 152.5) (end 210 117.5) (layer "Edge.Cuts") (width 0.1))
   (gr_line (start 210 62.5) (end 210 102.5) (layer "Edge.Cuts") (width 0.1))
   (gr_arc (start 210 102.5) (mid 209.899505 103.779901) (end 209.5 105) (layer "Edge.Cuts") (width 0.1))
   (gr_arc (start 209 113.5) (mid 208.288007 109.193412) (end 209.5 105) (layer "Edge.Cuts") (width 0.1))
-  (gr_line (start 110 153) (end 110 62.5) (layer "Edge.Cuts") (width 0.1))
+  (gr_line (start 110 152.5) (end 110 62.5) (layer "Edge.Cuts") (width 0.1))
   (gr_arc (start 110 62.5) (mid 111.464466 58.964466) (end 115 57.5) (layer "Edge.Cuts") (width 0.1))
-  (gr_arc (start 210 153) (mid 208.535534 156.535534) (end 205 158) (layer "Edge.Cuts") (width 0.1))
+  (gr_arc (start 210 152.5) (mid 208.535534 156.035534) (end 205 157.5) (layer "Edge.Cuts") (width 0.1))
   (gr_arc (start 209 113.5) (mid 209.735375 115.441156) (end 210 117.5) (layer "Edge.Cuts") (width 0.1))
   (gr_line (start 115 57.5) (end 205 57.5) (layer "Edge.Cuts") (width 0.1))
   (gr_arc (start 205 57.5) (mid 208.535534 58.964466) (end 210 62.5) (layer "Edge.Cuts") (width 0.1))
-  (via (at 203 156) (size 0.8) (drill 0.4) (layers "F.Cu" "B.Cu") (free) (net 2))
+  (via (at 202.5 156) (size 0.8) (drill 0.4) (layers "F.Cu" "B.Cu") (free) (net 2))
   (via (at 154 156) (size 0.8) (drill 0.4) (layers "F.Cu" "B.Cu") (free) (net 2))
   (via (at 204 67) (size 0.8) (drill 0.4) (layers "F.Cu" "B.Cu") (free) (net 2))
@@
   (via (at 113 96) (size 0.8) (drill 0.4) (layers "F.Cu" "B.Cu") (free) (net 2))
   (via (at 176 100) (size 0.8) (drill 0.4) (layers "F.Cu" "B.Cu") (free) (net 2))
-  (via (at 205 156) (size 0.8) (drill 0.4) (layers "F.Cu" "B.Cu") (free) (net 2))
+  (via (at 204.5 156) (size 0.8) (drill 0.4) (layers "F.Cu" "B.Cu") (free) (net 2))
   (via (at 142 120) (size 0.8) (drill 0.4) (layers "F.Cu" "B.Cu") (free) (net 2))
   (via (at 113 144) (size 0.8) (drill 0.4) (layers "F.Cu" "B.Cu") (free) (net 2))
@@
   (via (at 152 96) (size 0.8) (drill 0.4) (layers "F.Cu" "B.Cu") (free) (net 2))
   (via (at 206 67) (size 0.8) (drill 0.4) (layers "F.Cu" "B.Cu") (free) (net 2))
-  (via (at 207 156) (size 0.8) (drill 0.4) (layers "F.Cu" "B.Cu") (free) (net 2))
+  (via (at 206.5 156) (size 0.8) (drill 0.4) (layers "F.Cu" "B.Cu") (free) (net 2))
   (via (at 150 96) (size 0.8) (drill 0.4) (layers "F.Cu" "B.Cu") (free) (net 2))
   (via (at 171 120) (size 0.8) (drill 0.4) (layers "F.Cu" "B.Cu") (free) (net 2))
@@
     (connect_pads (clearance 0.508))
     (min_thickness 0.254) (filled_areas_thickness no)
-    (fill (thermal_gap 0.508) (thermal_bridge_width 0.508))
+    (fill yes (thermal_gap 0.508) (thermal_bridge_width 0.508))
     (polygon
       (pts
@@
     (connect_pads (clearance 0.508))
     (min_thickness 0.254) (filled_areas_thickness no)
-    (fill (thermal_gap 0.508) (thermal_bridge_width 0.508))
+    (fill yes (thermal_gap 0.508) (thermal_bridge_width 0.508))
     (polygon
       (pts

Commit message: Routed
Parts:
- added C12: 100nF, Capacitor_SMD:C_0603_1608Metric, F.Cu at (126.2, 104.4)
- added C13: 100nF, Capacitor_SMD:C_0603_1608Metric, F.Cu at (114.3, 124.9)
- added C14: 100nF, Capacitor_SMD:C_0603_1608Metric, F.Cu at (126.5, 124.9)
- added C15: 100nF, Capacitor_SMD:C_0603_1608Metric, F.Cu at (145.0, 124.9)
- added C16: 100nF, Capacitor_SMD:C_0603_1608Metric, F.Cu at (151.0, 153.3)
- added C17: 100nF, Capacitor_SMD:C_0603_1608Metric, F.Cu at (152.8, 153.3)
- added C18: 100nF, Capacitor_SMD:C_0603_1608Metric, F.Cu at (154.7, 153.3)
- added C19: 100nF, Capacitor_SMD:C_0603_1608Metric, F.Cu at (179.6, 94.8)
- added C20: 100nF, Capacitor_SMD:C_0603_1608Metric, F.Cu at (153.8, 103.9)
- added C21: 100nF, Capacitor_SMD:C_0603_1608Metric, F.Cu at (164.4, 113.1)
- added C22: 100nF, Capacitor_SMD:C_0603_1608Metric, F.Cu at (190.2, 127.0)
- added JP1: SolderJumper_2_Bridged, Jumper:SolderJumper-2_P1.3mm_Bridged_RoundedPad1.0x1.5mm, B.Cu at (165.9, 88.4)
- added JP2: SolderJumper_2_Bridged, Jumper:SolderJumper-2_P1.3mm_Bridged_RoundedPad1.0x1.5mm, B.Cu at (165.9, 82.3)
- added R10: 10k, Resistor_SMD:R_0603_1608Metric, F.Cu at (163.1, 81.5)
- added R9: 10k, Resistor_SMD:R_0603_1608Metric, F.Cu at (163.1, 85.7)
- moved C5 31.8 mm to (190.3, 132.9), turned to 0 degrees
- moved C3 21.7 mm to (190.3, 136.2), turned to 0 degrees
- moved C4 19.1 mm to (190.8, 147.0), turned to 0 degrees
- moved C7 0.45 mm to (201.3, 95.1)
Connections:
- D41 pad 3: GND -> unconnected-(D41-Pad3)
- U1 pad 19: unconnected-(U1-Pad19) -> Net-(R10-Pad1)
- U1 pad 20: unconnected-(U1-Pad20) -> Net-(R9-Pad1)
Routing:
- net +5V: track 0.00 -> 748.6 mm, vias 0 -> 13
- net +3V3: track 0.00 -> 150.9 mm, vias 0 -> 4
- net Net-(SW1-Pad2): track 0.00 -> 148.0 mm
- net /Buttons/row3: track 0.00 -> 128.1 mm, vias 0 -> 2
- net Net-(SW3-Pad3): track 0.00 -> 120.2 mm, vias 0 -> 2
- net Net-(SW10-Pad4): track 0.00 -> 112.7 mm, vias 0 -> 2
- net Net-(SW11-Pad4): track 0.00 -> 109.7 mm, vias 0 -> 4
- net Net-(SW10-Pad3): track 0.00 -> 105.8 mm, vias 0 -> 2
- net Net-(SW13-Pad12): track 0.00 -> 103.7 mm, vias 0 -> 2
- net /Buttons/col2: track 0.00 -> 97.8 mm, vias 0 -> 1
- net Net-(RV1-Pad2): track 0.00 -> 93.9 mm, vias 0 -> 1
- net /LEDs/DIN: track 0.00 -> 91.2 mm, vias 0 -> 1
- net Net-(SW13-Pad11): track 0.00 -> 89.8 mm, vias 0 -> 2
- net /Buttons/col5: track 0.00 -> 87.3 mm, vias 0 -> 5
- net /Buttons/row1: track 0.00 -> 84.3 mm
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
Commit message: Fixed ERC and DRC
Routing:
- net Net-(SW1-Pad2): track 148.0 -> 149.9 mm
- net GND: vias 199 -> 200
Changed lines of the file:
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@@
     (property "Sheetname" "LEDs")
     (attr smd)
-    (fp_text reference "D10" (at 1 3) (layer "F.SilkS")
+    (fp_text reference "D10" (at -1 2.8) (layer "F.SilkS")
       (effects (font (size 1 1) (thickness 0.15)))
     )
@@
   (via (at 133.3 62.3) (size 0.7) (drill 0.3) (layers "F.Cu" "B.Cu") (free) (net 2))
   (via (at 199.2 99.3) (size 0.7) (drill 0.3) (layers "F.Cu" "B.Cu") (free) (net 2))
+  (via (at 158.7 97.1) (size 0.7) (drill 0.3) (layers "F.Cu" "B.Cu") (free) (net 2))
   (via (at 145.7 75.1) (size 0.7) (drill 0.3) (layers "F.Cu" "B.Cu") (free) (net 2))
   (via (at 202.1 83.3) (size 0.7) (drill 0.3) (layers "F.Cu" "B.Cu") (free) (net 2))
@@
   (segment (start 202.1 58.4) (end 206.65 62.95) (width 0.25) (layer "F.Cu") (net 86))
   (segment (start 135.1 58.4) (end 202.1 58.4) (width 0.25) (layer "F.Cu") (net 86))
+  (segment (start 162.875489 99.924511) (end 160.449022 99.924511) (width 0.25) (layer "F.Cu") (net 87))
   (segment (start 139.65 106.1) (end 136.3 106.1) (width 0.25) (layer "F.Cu") (net 87))
   (segment (start 128.4 103) (end 127 103) (width 0.25) (layer "F.Cu") (net 87))
-  (segment (start 163.15 99.65) (end 162.875489 99.924511) (width 0.25) (layer "F.Cu") (net 87))
   (segment (start 196.5 93.3) (end 164.8 93.3) (width 0.25) (layer "F.Cu") (net 87))
-  (segment (start 159.1 96.9) (end 158.2 96.9) (width 0.25) (layer "F.Cu") (net 87))
   (segment (start 130.675489 107.924511) (end 127.775489 107.924511) (width 0.25) (layer "F.Cu") (net 87))
-  (segment (start 160 99.475489) (end 160 97.8) (width 0.25) (layer "F.Cu") (net 87))
   (segment (start 123.8 103) (end 121.65 105.15) (width 0.25) (layer "F.Cu") (net 87))
+  (segment (start 160 96.8) (end 159.2 96) (width 0.25) (layer "F.Cu") (net 87))
   (segment (start 127 103) (end 123.8 103) (width 0.25) (layer "F.Cu") (net 87))
   (segment (start 200.35 89.45) (end 196.5 93.3) (width 0.25) (layer "F.Cu") (net 87))
@@
   (segment (start 127.775489 107.924511) (end 127.5 107.649022) (width 0.25) (layer "F.Cu") (net 87))
   (segment (start 129.2 105.1) (end 129.2 103.8) (width 0.25) (layer "F.Cu") (net 87))
-  (segment (start 160.449022 99.924511) (end 160 99.475489) (width 0.25) (layer "F.Cu") (net 87))
   (segment (start 127 103) (end 127 100.7) (width 0.25) (layer "F.Cu") (net 87))
   (segment (start 136.3 106.1) (end 134.475489 107.924511) (width 0.25) (layer "F.Cu") (net 87))
-  (segment (start 146.1 106.1) (end 139.65 106.1) (width 0.25) (layer "F.Cu") (net 87))
-  (segment (start 158.2 96.9) (end 157.2 97.9) (width 0.25) (layer "F.Cu") (net 87))
   (segment (start 164.8 93.3) (end 163.15 94.95) (width 0.25) (layer "F.Cu") (net 87))
   (segment (start 129.2 103.8) (end 128.4 103) (width 0.25) (layer "F.Cu") (net 87))
-  (segment (start 160 97.8) (end 159.1 96.9) (width 0.25) (layer "F.Cu") (net 87))
+  (segment (start 160 99.475489) (end 160 96.8) (width 0.25) (layer "F.Cu") (net 87))
+  (segment (start 130.65 107.95) (end 130.675489 107.924511) (width 0.25) (layer "F.Cu") (net 87))
+  (segment (start 163.15 99.65) (end 162.875489 99.924511) (width 0.25) (layer "F.Cu") (net 87))
   (segment (start 157.2 99.7) (end 156.7 100.2) (width 0.25) (layer "F.Cu") (net 87))
-  (segment (start 130.65 107.95) (end 130.675489 107.924511) (width 0.25) (layer "F.Cu") (net 87))
-  (segment (start 156.7 100.2) (end 152 100.2) (width 0.25) (layer "F.Cu") (net 87))
+  (segment (start 158.2 96) (end 157.2 97) (width 0.25) (layer "F.Cu") (net 87))
+  (segment (start 146.1 106.1) (end 139.65 106.1) (width 0.25) (layer "F.Cu") (net 87))
+  (segment (start 159.2 96) (end 158.2 96) (width 0.25) (layer "F.Cu") (net 87))
   (segment (start 127 100.7) (end 127.5 100.2) (width 0.25) (layer "F.Cu") (net 87))
+  (segment (start 160.449022 99.924511) (end 160 99.475489) (width 0.25) (layer "F.Cu") (net 87))
   (segment (start 130.65 114.1) (end 130.65 107.95) (width 0.25) (layer "F.Cu") (net 87))
-  (segment (start 157.2 97.9) (end 157.2 99.7) (width 0.25) (layer "F.Cu") (net 87))
   (segment (start 163.15 94.95) (end 163.15 99.65) (width 0.25) (layer "F.Cu") (net 87))
   (segment (start 121.65 105.15) (end 121.65 106.1) (width 0.25) (layer "F.Cu") (net 87))
   (segment (start 130.65 99.35) (end 130.65 98.1) (width 0.25) (layer "F.Cu") (net 87))
   (segment (start 134.475489 107.924511) (end 130.675489 107.924511) (width 0.25) (layer "F.Cu") (net 87))
-  (segment (start 162.875489 99.924511) (end 160.449022 99.924511) (width 0.25) (layer "F.Cu") (net 87))
   (segment (start 127.5 107.649022) (end 127.5 106.1) (width 0.25) (layer "F.Cu") (net 87))
   (segment (start 127.5 106.1) (end 128.1 105.5) (width 0.25) (layer "F.Cu") (net 87))
   (segment (start 128.8 105.5) (end 129.2 105.1) (width 0.25) (layer "F.Cu") (net 87))
+  (segment (start 152 100.2) (end 146.1 106.1) (width 0.25) (layer "F.Cu") (net 87))
   (segment (start 128.1 105.5) (end 128.8 105.5) (width 0.25) (layer "F.Cu") (net 87))
   (segment (start 129.8 100.2) (end 130.65 99.35) (width 0.25) (layer "F.Cu") (net 87))
-  (segment (start 152 100.2) (end 146.1 106.1) (width 0.25) (layer "F.Cu") (net 87))
+  (segment (start 156.7 100.2) (end 152 100.2) (width 0.25) (layer "F.Cu") (net 87))
+  (segment (start 157.2 97) (end 157.2 99.7) (width 0.25) (layer "F.Cu") (net 87))
   (segment (start 170.3 91.7) (end 164 91.7) (width 0.25) (layer "F.Cu") (net 93))
   (segment (start 191.15 99.9) (end 191.15 98.45) (width 0.25) (layer "F.Cu") (net 93))

Commit message: Fixed ERC and DRC
Routing:
- net +5V: track 748.6 -> 747.7 mm
