File: pcb/leds.kicad_sch (KiCad schematic)
At the start: 62 parts

Commit message: Routed
Parts:
- added C12, C13, C14, C15, C16, C17, C18, C19, C20, C21, C22: 100nF, Capacitor_SMD:C_0603_1608Metric, symbol Device:C
Connections:
- net +5V: now also C12.1, C13.1, C14.1, C15.1, C16.1, C17.1, C18.1, C19.1, C20.1, C21.1, C22.1
- net GND: now also C12.2, C13.2, C14.2, C15.2, C16.2, C17.2, C18.2, C19.2, C20.2, C21.2, C22.2; no longer D41.3 (VSS)
Other:
- moved on the sheet: C1, C10, C11, C2, C3, C4, C5, C6, C7, C8, C9, D1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

Commit message: Fixed ERC and DRC
Connections:
- net GND: now also D41.3 (VSS)
Changed lines of the file:
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@@
     (pin "1")
   )
-  (symbol (lib_id "power:GND") (at 22.86 153.67 0) (unit 1)
+  (symbol (lib_id "power:GND") (at 22.86 151.13 0) (unit 1)
     (in_bom yes) (on_board yes) (fields_autoplaced)
-    (property "Reference" "#PWR092" (id 0) (at 22.86 160.02 0)
+    (property "Reference" "#PWR092" (id 0) (at 22.86 157.48 0)
       (effects (font (size 1.27 1.27)) hide)
     )
-    (property "Value" "GND" (id 1) (at 22.86 158.75 0))
-    (property "Footprint" "" (id 2) (at 22.86 153.67 0)
+    (property "Value" "GND" (id 1) (at 22.86 156.21 0))
+    (property "Footprint" "" (id 2) (at 22.86 151.13 0)
       (effects (font (size 1.27 1.27)) hide)
     )
-    (property "Datasheet" "" (id 3) (at 22.86 153.67 0)
+    (property "Datasheet" "" (id 3) (at 22.86 151.13 0)
       (effects (font (size 1.27 1.27)) hide)
     )

Commit message: Fixed ERC and DRC
Parts:
- C1, C10, C11, C12, C13, C14, C15, C16, C17, C18, C19, C2, C20, C21, C22, C3, C4, C5, C6, C7, C8, C9: LCSC (none) -> C14663
- D1, D10, D11, D12, D13, D14, D15, D16, D17, D18, D19, D2, D20, D21, D22, D23, D24, D25, D26, D27, D28, D29, D3, D30, D31, D32, D33, D34, D35, D36, D37, D38, D39, D4, D40, D41, D42, D43, D44, D45, D46, D47, D48, D49, D5, D50, D51, D6, D7, D8, D9: LCSC (none) -> C2890364
